File: SSB Amplifier.kicad_pcb (KiCad board)
At the start: 2 copper layers, 85.8 x 51 mm, 32 parts, among them J1 PCB_SMA, J2 BNC, J3 Pad, J4 Pad, Q1 2N3904, Q2 2SC5706, Q3 2SC5706, U1 MCP1703A-5002_SOT223

Commit message: gg
Parts:
- added C11: .1uF, Xenir:Capacitor 0805, F.Cu at (100.3, 106.2)
- added R11: 10k, Xenir:Resistor 0805, F.Cu at (98.2, 103.7)
- added R12: 10k, Xenir:Resistor 0805, F.Cu at (98.2, 108.2)
- Q1: value 2N3904 -> 2N3904-SMD
- R4: value 1k -> 10k
- moved R2 5.08 mm to (114.0, 103.3), turned to 270 degrees
- moved Q1 1.84 mm to (104.5, 106.2), turned to 90 degrees
- moved R1 1.12 mm to (106.6, 107.7)
Connections:
- J1 pad 1: Net-(J1-Pad1) -> Net-(C11-Pad1)
- Q1 pad 1: Net-(C1-Pad1) -> Net-(C11-Pad2)
- Q1 pad 2: Net-(J1-Pad1) -> Net-(C1-Pad1)
Routing:
- net Net-(J1-Pad1): track 19.9 -> 0.00 mm, vias 1 -> 0
- net Net-(C11-Pad2): track 0.00 -> 8.53 mm
- net Net-(C11-Pad1): track 0.00 -> 7.82 mm, vias 0 -> 1
- net +5V: track 22.3 -> 25.1 mm
- net Net-(C1-Pad1): track 11.6 -> 8.89 mm
- net Net-(C1-Pad2): track 15.2 -> 12.4 mm
- net Net-(C2-Pad1): track 10.8 -> 8.33 mm

Commit message: gg
Parts:
- R5: value 1k -> 10
Changed lines of the file:
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@@
   )
   (setup
-    (last_trace_width 1)
+    (last_trace_width 0.25)
     (user_trace_width 0.5)
     (user_trace_width 1)
@@
       (effects (font (size 0.5 0.5) (thickness 0.125)))
     )
-    (fp_text value 1k (at 0 1) (layer F.Fab)
-      (effects (font (size 0.5 0.5) (thickness 0.125)))
-    )
+    (fp_text value 10 (at 0 1) (layer F.Fab)
+      (effects (font (size 0.5 0.5) (thickness 0.125)))
+    )
