File: SSB Amplifier.sch (KiCad schematic (older format))
At the start: 32 parts, among them J1 PCB_SMA, J2 BNC, J3 Pad, J4 Pad, Q1 2N3904, Q2 2SC5706, Q3 2SC5706, U1 MCP1703A-5002_SOT223

Commit message: gg
Parts:
- removed Q1: 2N3904, Package_TO_SOT_SMD:SOT-23, symbol Transistor_BJT:2N3904
- added C11: .1uF, Xenir:Capacitor 0805, symbol Xenir:Capacitor
- added Q1: 2N3904-SMD, Package_TO_SOT_SMD:SOT-23, symbol Xenir:2N3904-SMD
- added R11, R12: 10k, Xenir:Resistor 0805, symbol Xenir:Resistor
- R4: value 1k -> 10k
Connections:
- net +5V: now also Q1.3 (C), R11.2
- net GND: now also R12.1
- net at C1.1, R1.1: now also Q1.2 (E)
- net at J1.1: now also C11.1
- new net: C11.2, Q1.1 (B), R11.1, R12.2
Other:
- moved on the sheet: J1
Changed lines of the file:
@@
 $EndDescr
-$Comp
-L Transistor_BJT:2N3904 Q1
-U 1 1 5F4B87C2
-P 2900 3350
-F 0 "Q1" H 3100 3425 50  0000 L CNN
-F 1 "2N3904" H 3100 3350 50  0000 L CNN
-F 2 "Package_TO_SOT_SMD:SOT-23" H 3100 3275 50  0001 L CIN
-F 3 "https://www.fairchildsemi.com/datasheets/2N/2N3904.pdf" H 2900 3350 50  0001 L CNN
-	1    2900 3350
-	1    0    0    -1
-$EndComp
 $Comp
 L Xenir:Resistor R1
@@
 	1    0    0    -1
 $EndComp
-Connection ~ 3000 3550
 $Comp
 L power:GND #PWR0101
@@
 L Xenir:PCB_SMA J1
 U 1 1 5F4BBF58
-P 2200 3150
-F 0 "J1" H 2250 3050 50  0000 C CNN
-F 1 "PCB_SMA" H 2200 3150 50  0000 C CNN
-F 2 "Xenir:PCB SMA" H 2200 3150 50  0001 C CNN
-F 3 "" H 2200 3150 50  0001 C CNN
-	1    2200 3150
+P 1800 3150
+F 0 "J1" H 1850 3050 50  0000 C CNN
+F 1 "PCB_SMA" H 1800 3150 50  0000 C CNN
+F 2 "Xenir:PCB SMA" H 1800 3150 50  0001 C CNN
+F 3 "" H 1800 3150 50  0001 C CNN
+	1    1800 3150
 	1    0    0    -1
 $EndComp
@@
 L power:GND #PWR0103
 U 1 1 5F4BD3BA
-P 2300 3450
-F 0 "#PWR0103" H 2300 3200 50  0001 C CNN
-F 1 "GND" H 2300 3300 50  0000 C CNN
-F 2 "" H 2300 3450 50  0001 C CNN
-F 3 "" H 2300 3450 50  0001 C CNN
-	1    2300 3450
-	1    0    0    -1
-$EndComp
-Wire Wire Line
-	2300 3350 2700 3350
+P 1900 3450
+F 0 "#PWR0103" H 1900 3200 50  0001 C CNN
+F 1 "GND" H 1900 3300 50  0000 C CNN
+F 2 "" H 1900 3450 50  0001 C CNN
+F 3 "" H 1900 3450 50  0001 C CNN
+	1    1900 3450
+	1    0    0    -1
+$EndComp
 $Comp
 L Xenir:Resistor R2
@@
 P 3900 2750
 F 0 "R4" H 3900 2825 28  0000 C CNN
-F 1 "1k" H 3900 2675 28  0000 C CNN
+F 1 "10k" H 3900 2675 28  0000 C CNN
 F 2 "Xenir:Resistor 0805" H 3900 2650 50  0001 C CNN
 F 3 "" H 3900 2650 50  0001 C CNN
@@
 	1    0    0    -1
 $EndComp
+$Comp
+L Xenir:2N3904-SMD Q1
+U 1 1 5F4C610F
+P 2900 3350
+F 0 "Q1" H 3100 3425 50  0000 L CNN
+F 1 "2N3904-SMD" H 3100 3350 50  0000 L CNN
+F 2 "Package_TO_SOT_SMD:SOT-23" H 3100 3275 50  0001 L CIN
+F 3 "https://www.fairchildsemi.com/datasheets/2N/2N3904.pdf" H 2900 3350 50  0001 L CNN
+	1    2900 3350
+	1    0    0    -1
+$EndComp
+Connection ~ 3000 3550
+$Comp
+L Xenir:Resistor R11
+U 1 1 5F4C8B82
+P 2700 3150
+F 0 "R11" H 2700 3225 28  0000 C CNN
+F 1 "10k" H 2700 3075 28  0000 C CNN
+F 2 "Xenir:Resistor 0805" H 2700 3050 50  0001 C CNN
+F 3 "" H 2700 3050 50  0001 C CNN
+	1    2700 3150
+	0    -1   -1   0
+$EndComp
+$Comp
+L Xenir:Resistor R12
+U 1 1 5F4CA41C
+P 2700 3550
+F 0 "R12" H 2700 3625 28  0000 C CNN
+F 1 "10k" H 2700 3475 28  0000 C CNN
+F 2 "Xenir:Resistor 0805" H 2700 3450 50  0001 C CNN
+F 3 "" H 2700 3450 50  0001 C CNN
+	1    2700 3550
+	0    -1   -1   0
+$EndComp
+Connection ~ 2700 3350
+$Comp
+L power:GND #PWR0122
+U 1 1 5F4CAC87
+P 2700 3750
+F 0 "#PWR0122" H 2700 3500 50  0001 C CNN
+F 1 "GND" H 2700 3600 50  0000 C CNN
+F 2 "" H 2700 3750 50  0001 C CNN
+F 3 "" H 2700 3750 50  0001 C CNN
+	1    2700 3750
+	1    0    0    -1
+$EndComp
+$Comp
+L power:+5V #PWR0123
+U 1 1 5F4CB4F5
+P 2700 2950
+F 0 "#PWR0123" H 2700 2800 50  0001 C CNN
+F 1 "+5V" H 2700 3090 50  0000 C CNN
+F 2 "" H 2700 2950 50  0001 C CNN
+F 3 "" H 2700 2950 50  0001 C CNN
+	1    2700 2950
+	1    0    0    -1
+$EndComp
+$Comp
+L Xenir:Capacitor C11
+U 1 1 5F4CB9B7
+P 2550 3350
+F 0 "C11" H 2550 3475 28  0000 C CNN
+F 1 ".1uF" H 2550 3225 28  0000 C CNN
+F 2 "Xenir:Capacitor 0805" H 2550 3200 50  0001 C CNN
+F 3 "" H 2550 3200 50  0001 C CNN
+	1    2550 3350
+	1    0    0    -1
+$EndComp
+Wire Wire Line
+	1900 3350 2400 3350
 $EndSCHEMATC

Commit message: gg
Parts:
- R5: value 1k -> 10
Changed lines of the file:
@@
 P 4300 3750
 F 0 "R5" H 4300 3825 28  0000 C CNN
-F 1 "1k" H 4300 3675 28  0000 C CNN
+F 1 "10" H 4300 3675 28  0000 C CNN
 F 2 "Xenir:Resistor 0805" H 4300 3650 50  0001 C CNN
 F 3 "" H 4300 3650 50  0001 C CNN
